File: PCB/WateringSystem.kicad_pcb (KiCad board)
At the start: 2 copper layers, 99.6 x 72.1 mm, 47 parts, among them J1 Jack-DC, J2 Conn_01x02, J3 Conn_01x02, J4 Conn_01x04, J5 Conn_01x04, J6 Conn_01x04, J7 Conn_01x04, Q1 Q_NMOS_GDS, Q2 Q_NMOS_GDS, Q3 Q_NMOS_GDS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

Commit message: CLion project files
Parts:
- moved C3 1.51 mm to (73.0, 120.8)
- moved C4 1.51 mm to (73.0, 128.3)
Routing:
- net +5V: track 34.3 -> 28.2 mm
Changed lines of the file:
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@@
   )
   (setup
-    (last_trace_width 0.25)
+    (last_trace_width 1)
     (user_trace_width 0.5)
     (user_trace_width 1)
@@
   )
   (module Capacitors_ThroughHole:C_Radial_D5_L6_P2.5 (layer F.Cu)
-    (at 74.47 120.84)
+    (at 72.96 120.78)
     (descr "Radial Electrolytic Capacitor Diameter 5mm x Length 6mm, Pitch 2.5mm")
     (tags "Electrolytic Capacitor")
@@
   )
   (module Capacitors_ThroughHole:C_Radial_D5_L6_P2.5 (layer F.Cu)
-    (at 74.5 127.89)
+    (at 73.04 128.28)
     (descr "Radial Electrolytic Capacitor Diameter 5mm x Length 6mm, Pitch 2.5mm")
     (tags "Electrolytic Capacitor")
@@
   (gr_line (start 59.9 75.75) (end 134.51 75.75) (layer Edge.Cuts) (width 0.15))
   (segment (start 123.82 108.09) (end 123.83 108.08) (width 0.25) (layer F.Cu) (net 0))
-  (segment (start 74.47 120.84) (end 74.47 124.03) (width 1) (layer F.Cu) (net 1))
+  (segment (start 72.74 127.98) (end 70.52 127.98) (width 1) (layer F.Cu) (net 1))
+  (via (at 70.52 127.98) (size 0.6) (drill 0.4) (layers F.Cu B.Cu) (net 1))
+  (segment (start 70.52 127.98) (end 67.93 130.57) (width 1) (layer B.Cu) (net 1))
+  (segment (start 67.93 130.57) (end 65.04 130.57) (width 1) (layer B.Cu) (net 1))
+  (via (at 65.04 130.57) (size 0.6) (drill 0.4) (layers F.Cu B.Cu) (net 1))
+  (segment (start 65.04 130.57) (end 58.48 124.01) (width 1) (layer F.Cu) (net 1))
+  (segment (start 58.48 124.01) (end 58.48 120.4) (width 1) (layer F.Cu) (net 1))
+  (segment (start 58.48 120.4) (end 56.44 118.36) (width 1) (layer F.Cu) (net 1))
   (segment (start 56.44 118.36) (end 53.21 118.36) (width 1) (layer F.Cu) (net 1))
-  (segment (start 58.48 120.4) (end 56.44 118.36) (width 1) (layer F.Cu) (net 1))
-  (segment (start 58.48 124.01) (end 58.48 120.4) (width 1) (layer F.Cu) (net 1))
-  (segment (start 65.04 130.57) (end 58.48 124.01) (width 1) (layer F.Cu) (net 1))
-  (via (at 65.04 130.57) (size 0.6) (drill 0.4) (layers F.Cu B.Cu) (net 1))
-  (segment (start 67.93 130.57) (end 65.04 130.57) (width 1) (layer B.Cu) (net 1))
-  (segment (start 70.52 127.98) (end 67.93 130.57) (width 1) (layer B.Cu) (net 1))
-  (via (at 70.52 127.98) (size 0.6) (drill 0.4) (layers F.Cu B.Cu) (net 1))
-  (segment (start 74.47 124.03) (end 70.52 127.98) (width 1) (layer F.Cu) (net 1))
+  (segment (start 72.74 127.98) (end 73.04 128.28) (width 1) (layer F.Cu) (net 1))
   (segment (start 142.4 112.96) (end 142.4 114.23) (width 1) (layer B.Cu) (net 2))
   (segment (start 142.4 114.23) (end 137.9 118.73) (width 1) (layer B.Cu) (net 2))

Commit message: fixed screen connector on PCB
Parts:
- added REF**: 1pin, Connect:1pin, F.Cu at (119.9, 90.7)
- J2, J3: moved to B.Cu
- moved TFT1 17.7 mm to (74.2, 105.6), turned to 180 degrees
- moved J3 0.11 mm to (141.6, 123.6), turned to 180 degrees
- moved J2 0.05 mm to (68.3, 142.2), turned to 90 degrees
Routing:
- net GND: track 88.7 -> 112.0 mm
- net Net-(LS1-Pad6): track 11.1 -> 27.2 mm, vias 0 -> 1
- net Net-(LS1-Pad11): track 21.7 -> 31.8 mm
- net Net-(LS1-Pad15): track 26.8 -> 16.8 mm, vias 0 -> 1
- net Net-(LS1-Pad10): track 8.47 -> 18.3 mm, vias 0 -> 1
- net Net-(LS1-Pad12): track 11.8 -> 21.0 mm, vias 0 -> 1
- net Net-(LS1-Pad9): track 17.9 -> 23.2 mm
- net Net-(C5-Pad2): track 91.2 -> 87.1 mm
- net Net-(LS1-Pad2): track 30.0 -> 27.5 mm, vias 0 -> 1
- net Net-(D3-Pad1): track 74.9 -> 72.7 mm
- net Net-(LS1-Pad14): track 27.3 -> 29.4 mm, vias 1 -> 0
- net Net-(LS1-Pad4): track 29.7 -> 28.6 mm, vias 0 -> 1
- net Net-(LS1-Pad7): track 22.3 -> 23.1 mm
Other:
- board text added: "- +"
- board text added: "Arduino"
- board text added: "Coils"
- board text added: "Plant Watering System v1.1"
- board text removed: "Plant Watering System v1.0"

Commit message: fixed and updated PCB
Parts:
- added Q5: Q_NMOS_GDS, TO_SOT_Packages_THT:TO-220_Vertical, B.Cu at (63.3, 113.5)
- added R13: 1k, Resistors_SMD:R_1206_HandSoldering, F.Cu at (64.8, 119.6)
- added R14: 10k, Resistors_SMD:R_1206_HandSoldering, F.Cu at (61.2, 119.6)
- moved D_COIL_1 2.11 mm to (84.8, 124.1)
- moved D_COIL_2 2.11 mm to (93.9, 123.9)
- moved D_COIL_3 2.11 mm to (103.1, 124.0)
- moved D_COIL_4 2.11 mm to (112.1, 124.1)
- moved J4 1.52 mm to (88.8, 125.5)
- moved J5 1.52 mm to (97.8, 125.5)
- moved J6 1.52 mm to (106.8, 125.5)
- moved J7 1.52 mm to (115.8, 125.5)
- moved TFT1 1.51 mm to (74.2, 107.2)
Connections:
- J4 pad 1: GND -> Net-(J4-Pad1)
- J5 pad 1: GND -> Net-(J4-Pad1)
- J6 pad 1: GND -> Net-(J4-Pad1)
- J7 pad 1: GND -> Net-(J4-Pad1)
- R1 pad 1: Net-(R1-Pad1) -> +5V
- R2 pad 1: Net-(R1-Pad1) -> +5V
- R3 pad 1: Net-(R1-Pad1) -> +5V
- R4 pad 1: Net-(R1-Pad1) -> +5V
- U1 pad 30: Net-(R1-Pad1) -> Net-(R13-Pad1)
Routing:
- net Net-(J4-Pad1): track 0.00 -> 93.6 mm, vias 0 -> 1
- net +5V: track 28.2 -> 67.1 mm
- net Net-(R13-Pad1): track 0.00 -> 33.2 mm
- net Net-(R1-Pad1): track 16.6 -> 0.00 mm
- net GND: track 112.0 -> 122.4 mm, vias 5 -> 6
- net Net-(Q5-Pad1): track 0.00 -> 8.49 mm
- net Net-(D3-Pad1): track 72.7 -> 67.3 mm
- net Net-(R10-Pad1): track 40.5 -> 44.0 mm
- net Net-(R12-Pad1): track 54.1 -> 57.2 mm
- net Net-(J4-Pad4): track 68.4 -> 70.6 mm
- net Net-(J7-Pad4): track 118.5 -> 116.6 mm
- net Net-(R8-Pad1): track 28.7 -> 30.6 mm
- net Net-(LS1-Pad4): track 28.6 -> 29.9 mm
- net Net-(LS1-Pad2): track 27.5 -> 28.9 mm
- net Net-(LS1-Pad6): track 27.2 -> 28.5 mm
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